File: coil-board/coil-board.kicad_pcb (KiCad board)
At the start: 2 copper layers, 0 parts

Commit message: Add coil and solder pad to coil board
Parts:
- added ?: , clipboard:f60c125d-a46e-4052-9ba0-15b3719510b7, F.Cu at (71.0, 129.0)
- added ?: , clipboard:f60c125d-a46e-4052-9ba0-15b3719510b7, F.Cu at (101.8, 148.3)
- added ?: , clipboard:f60c125d-a46e-4052-9ba0-15b3719510b7, F.Cu at (129.0, 129.0)
- added ?: , clipboard:f60c125d-a46e-4052-9ba0-15b3719510b7, F.Cu at (98.2, 148.3)
- added REF**: MountingHole_2.1mm, MountingHole:MountingHole_2.1mm, F.Cu at (78.0, 122.0)
- added REF**: MountingHole_2.1mm, MountingHole:MountingHole_2.1mm, F.Cu at (122.0, 122.0)
- added REF**: MountingHole_2.1mm, MountingHole:MountingHole_2.1mm, F.Cu at (78.0, 78.0)
- added REF**: MountingHole_2.1mm, MountingHole:MountingHole_2.1mm, F.Cu at (122.0, 78.0)
Routing:
- net (no net): track 0.00 -> 14068.7 mm
Other:
- board outline added: 100 x 100 mm
